File: GlowTubePCB/GlowTube.kicad_pcb (KiCad board)
At the start: 2 copper layers, 139.7 x 145.5 mm, 28 parts, among them Q1 MMBT2222A, Q2 MMBT2222A, U1 ESP32-WROOM-32E (4MB), U2 PW14, U3 BL1117-33CX, U4 Val**

Commit message: added qr code to pcb
Other:
- board text added: "PCB files: https://bit.ly/3srVD59"
- board text removed: "PCB files: https://bit.ly/...."

Commit message: added GlowTube v1.0 beta 1
Parts:
- added C10: 1uF, Capacitor_SMD:C_0603_1608Metric_Pad1.08x0.95mm_HandSolder, F.Cu at (118.2, 162.8)
- added J1: Conn_01x08, Connector_PinSocket_2.54mm:PinSocket_1x08_P2.54mm_Vertical, F.Cu at (89.5, 136.0)
- added LED2: LED_strip_contact_pads, Connector:LED strip connector pad, B.Cu at (159.3, 82.3)
- added Q3: AP40P05, Package_TO_SOT_SMD:SOT-23, F.Cu at (137.2, 131.8)
- added Q4: AP40P05, Package_TO_SOT_SMD:SOT-23, F.Cu at (129.8, 135.4)
- added R7: 10K, Resistor_SMD:R_0603_1608Metric_Pad0.98x0.95mm_HandSolder, F.Cu at (114.1, 162.8)
- added RJ1: R-RJ11R06P-A800, R-RJ11R06P-A800:R-RJ11R06P-A800, F.Cu at (104.0, 159.7)
- added SW1: SW-SMD_4P-L3.7-W3.0-P1.50-LS4.7, TS-1185EC-C-D-B:TS-1185EC-C-D-B, F.Cu at (123.7, 160.4)
- added SW2: SW-SMD_4P-L3.7-W3.0-P1.50-LS4.7, TS-1185EC-C-D-B:TS-1185EC-C-D-B, F.Cu at (116.2, 160.4)
- moved R1 58.1 mm to (159.3, 85.7), turned to 90 degrees
- moved LED1 54.6 mm to (159.2, 82.3), turned to 0 degrees
- moved R2 38.3 mm to (98.5, 148.5)
- moved REF** 38.1 mm to (123.7, 144.8)
- moved Q2 37.6 mm to (142.6, 143.1)
- moved Q1 37.6 mm to (139.0, 143.2)
- moved R4 37.6 mm to (140.7, 146.0)
- moved R5 37.6 mm to (140.8, 140.2)
- moved G*** 37.6 mm to (134.2, 145.1)
- moved G*** 37.3 mm to (134.3, 129.3)
- moved MK1 36.8 mm to (140.9, 105.9), turned to -90 degrees
- moved R3 34.7 mm to (100.3, 148.5)
- moved R6 33.3 mm to (144.5, 106.0), turned to 90 degrees
- moved C8 33.1 mm to (140.4, 103.0), turned to 180 degrees
- moved U1 32.6 mm to (146.8, 119.2)
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Connections:
- C3 pad 2: USB-C 5V -> +5V
- C7 pad 2: +3V3 -> Net-(C7-Pad2)
- F1 pad 2: USB-C 5V -> +5V
- U1 pad 9: IO33 -> IO33/TESTBUTTON
- U2 pad 1: IO16/LED1 -> LED1 DATA IN
- U3 pad 2: +3V3 -> Net-(C7-Pad2)
- U3 pad 3: USB-C 5V -> +5V
- U3 pad 4: +3V3 -> Net-(C7-Pad2)
- U4 pad 8: USB-C 5V -> +5V
Routing:
- net GND: track 0.00 -> 427.0 mm, vias 0 -> 9
- net +5V: track 0.00 -> 172.1 mm, vias 0 -> 5
- net +3V3: track 0.00 -> 147.3 mm, vias 0 -> 6
- net LED1 DATA IN: track 0.00 -> 99.4 mm, vias 0 -> 2
- net RESET: track 0.00 -> 89.6 mm, vias 0 -> 3
- net IO25/A1/DAC1: track 0.00 -> 86.5 mm, vias 0 -> 2
- net IO26/A0/DAC2: track 0.00 -> 86.3 mm, vias 0 -> 2
- net IO33/TESTBUTTON: track 0.00 -> 78.0 mm, vias 0 -> 4
- net IO5: track 0.00 -> 59.7 mm, vias 0 -> 2
- net IO13: track 0.00 -> 57.8 mm, vias 0 -> 2
- net IO12: track 0.00 -> 56.7 mm, vias 0 -> 2
- net USB-C DATA+: track 0.00 -> 56.1 mm, vias 0 -> 4
- net USB-C DATA-: track 0.00 -> 54.4 mm, vias 0 -> 2
- net RECEIVER 5V: track 0.00 -> 47.6 mm, vias 0 -> 1
- net TXD0: track 0.00 -> 34.7 mm
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Other:
- board size 139.7 x 145.5 mm -> 87.3 x 86.3 mm
- board text added: "5V"
- board text added: "GND"
- board text added: "IO12/MISO IO13/MOSI IO5 IO25/A1 IO26/A0 3.3V GND 5V"
- board text added: "LED 1 (IO16)"
- board text added: "RESET"
- board text added: "TEST"
- board text added: "v1.0 beta 1"
- board text removed: "5V D GND"
- board text removed: "v0.1"
